Commit message: cleaning up xacro and launch files to suit robot

File: src/mobile_robot_2wd_description/urdf/robot_model.xacro (robot description, xacro)
@@ -7,4 +7,7 @@
   <xacro:property name="M_PI_2" value="1.570796327" />
   <xacro:property name="DEG_TO_RAD" value="0.017453293" />
+  <material name="black">
+    <color rgba="0 0 0 1"/>
+  </material>
  <!-- <xacro:macro name="mobile_robot">   -->
     <link name="base_footprint"/>
@@ -48,5 +51,5 @@
 <!-- Wheel and caster wheel link  -->
         <!-- NOTE This may prevent gazebo from working with this model -->
-	  <joint name="left_wheel_joint" type="fixed">
+	  <joint name="left_wheel_joint" type="continuous">
 	    <origin xyz="-0.06 0 0" rpy="0 0 0"/>
 	    <parent link="base_link"/>
@@ -100,5 +103,5 @@
         <!-- Fixed because we never rotate it anyway, it is just for show -->
         <!-- NOTE This may prevent gazebo from working with this model -->
-	  <joint name="right_wheel_joint" type="fixed">
+	  <joint name="right_wheel_joint" type="continuous">
 	    <origin xyz="0.06 0 0" rpy="0 0 0"/>
 	    <parent link="base_link"/>
@@ -106,5 +109,4 @@
 	    <axis xyz="1 0 0"/>
 	  </joint>
-<!--
     <joint name="caster_front_joint" type="fixed">
       <parent link="base_link"/>
@@ -127,5 +129,4 @@
       </inertial>
     </link>
--->
     <joint name="robot_caster_back_joint" type="fixed">
       <parent link="base_link"/>
@@ -150,5 +151,5 @@
 	      <origin xyz="0 0 0" rpy="0 ${M_PI/2} 0" />
 	      <geometry>
-            		<cylinder radius="0.01" length = "0.1"/>
+            	<cylinder radius="0.01" length = "0.1"/>
 	      </geometry>
 	    </collision>
